Commit message: added velocity control to the robot control. The inverse kinematic is found in th epanda_velocity_controller.

File: panda_ws/src/panda_description/urdf/gazebo.xacro (robot description, xacro)
@@ -17,10 +17,15 @@
     </xacro:unless>
     <!-- Joint 1 -->
-    <joint name="panda_joint1">
+     <joint name="panda_joint1">
       <command_interface name="position">
         <param name="min">-2.9671</param>
         <param name="max">2.9671</param>
       </command_interface>
+      <command_interface name="velocity">
+        <param name="min">-10.0</param>
+        <param name="max">10.0</param>
+      </command_interface>
       <state_interface name="position"/>
+      <state_interface name="velocity"/>
     </joint>
     <!-- Joint 2 -->
@@ -30,5 +35,10 @@
         <param name="max">1.8326</param>
       </command_interface>
+      <command_interface name="velocity">
+        <param name="min">-10.0</param>
+        <param name="max">10.0</param>
+      </command_interface>
       <state_interface name="position"/>
+      <state_interface name="velocity"/>
     </joint>
     <!-- Joint 3 -->
@@ -38,5 +48,10 @@
         <param name="max">2.9671</param>
       </command_interface>
+      <command_interface name="velocity">
+        <param name="min">-10.0</param>
+        <param name="max">10.0</param>
+      </command_interface>
       <state_interface name="position"/>
+      <state_interface name="velocity"/>
     </joint>
     <!-- Joint 4 -->
@@ -46,5 +61,10 @@
         <param name="max">0.0</param>
       </command_interface>
+      <command_interface name="velocity">
+        <param name="min">-10.0</param>
+        <param name="max">10.0</param>
+      </command_interface>
       <state_interface name="position"/>
+      <state_interface name="velocity"/>
     </joint>
     <!-- Joint 5 -->
@@ -54,5 +74,10 @@
         <param name="max">2.9671</param>
       </command_interface>
+      <command_interface name="velocity">
+        <param name="min">-10.0</param>
+        <param name="max">10.0</param>
+      </command_interface>
       <state_interface name="position"/>
+      <state_interface name="velocity"/>
     </joint>
     <!-- Joint 6 -->
@@ -62,5 +87,10 @@
         <param name="max">3.8223</param>
       </command_interface>
+      <command_interface name="velocity">
+        <param name="min">-10.0</param>
+        <param name="max">10.0</param>
+      </command_interface>
       <state_interface name="position"/>
+      <state_interface name="velocity"/>
     </joint>
     <!-- Joint 7 -->
@@ -70,5 +100,10 @@
         <param name="max">2.9671</param>
       </command_interface>
+      <command_interface name="velocity">
+        <param name="min">-10.0</param>
+        <param name="max">10.0</param>
+      </command_interface>
       <state_interface name="position"/>
+      <state_interface name="velocity"/>
     </joint>
     <!-- Gripper Finger Joint 1 -->
