Commit message: removed the old gripper and added a simple tool to represent a probe in the eye

File: panda_ws/src/panda_description/urdf/arm.xacro (robot description, xacro)
@@ -216,82 +216,60 @@
     <limit effort="30.0" lower="-2.9671" upper="2.9671" velocity="10.0"/>
   </joint>
-  <!-- Hand Link -->
-  <link name="panda_hand">
-    <visual>
-      <geometry>
-        <mesh filename="package://panda_description/meshes/visual/hand.dae"/>
-      </geometry>
-    </visual>
-    <collision>
-      <geometry>
-        <mesh filename="package://panda_description/meshes/collision/hand.obj"/>
-      </geometry>
-    </collision>
-      <inertial>
-          <origin xyz="0 0 0" rpy="0.0 0.0 0.0"/>
-          <mass value="0.1"/>
-          <inertia ixx="0.1" ixy="0.0" ixz="0.0" iyy="0.1" iyz="0.0" izz="0.1"/>
-      </inertial>
-  </link>
-  <!-- Hand Joint -->
-  <joint name="panda_hand_joint" type="fixed">
+  <!-- Tool Link: simple probe (two cylinders) -->
+  <link name="panda_tool">
+    <visual>
+      <origin xyz="0 0 0.02" rpy="0 0 0"/>
+      <geometry>
+        <cylinder radius="0.025" length="0.04"/>
+      </geometry>
+    </visual>
+    <visual>
+      <origin xyz="0 0 0.05" rpy="0 0 0"/>
+      <geometry>
+        <cylinder radius="0.0025" length="0.1"/>
+      </geometry>
+    </visual>
+    <visual>
+      <origin xyz="0 0 0.11" rpy="0 0 0"/>
+      <geometry>
+        <cylinder radius="0.0008" length="0.02"/>
+      </geometry>
+    </visual>
+    <collision>
+      <origin xyz="0 0 0.02" rpy="0 0 0"/>
+      <geometry>
+        <cylinder radius="0.025" length="0.04"/>
+      </geometry>
+    </collision>
+    <collision>
+      <origin xyz="0 0 0.05" rpy="0 0 0"/>
+      <geometry>
+        <cylinder radius="0.0025" length="0.1"/>
+      </geometry>
+    </collision>
+    <collision>
+      <origin xyz="0 0 0.11" rpy="0 0 0"/>
+      <geometry>
+        <cylinder radius="0.0008" length="0.02"/>
+      </geometry>
+    </collision>
+    <inertial>
+      <origin xyz="0 0 0.04" rpy="0 0 0"/>
+      <mass value="0.05"/>
+      <inertia ixx="0.0001" ixy="0.0" ixz="0.0" iyy="0.0001" iyz="0.0" izz="0.0001"/>
+    </inertial>
+  </link>
+  <!-- Tool joint at flange -->
+  <joint name="panda_tool_joint" type="fixed">
     <parent link="panda_link7"/>
-    <child link="panda_hand"/>
-    <origin rpy="0 0 -0.785398163397" xyz="0 0 0.106"/>
-  </joint>
-  <!-- Left Finger Link -->
-  <link name="panda_leftfinger">
-    <visual>
-      <geometry>
-        <mesh filename="package://panda_description/meshes/visual/finger.dae"/>
-      </geometry>
-    </visual>
-    <collision>
-      <geometry>
-        <mesh filename="package://panda_description/meshes/collision/finger.obj"/>
-      </geometry>
-    </collision>
-      <inertial>
-          <origin xyz="0 0 0" rpy="0.0 0.0 0.0"/>
-          <mass value="0.1"/>
-          <inertia ixx="0.1" ixy="0.0" ixz="0.0" iyy="0.1" iyz="0.0" izz="0.1"/>
-      </inertial>
-  </link>
-  <!-- Right Finger Link -->
-  <link name="panda_rightfinger">
-    <visual>
-      <origin rpy="0 0 3.14159265359" xyz="0 0 0"/>
-      <geometry>
-        <mesh filename="package://panda_description/meshes/visual/finger.dae"/>
-      </geometry>
-    </visual>
-    <collision>
-      <origin rpy="0 0 3.14159265359" xyz="0 0 0"/>
-      <geometry>
-        <mesh filename="package://panda_description/meshes/collision/finger.obj"/>
-      </geometry>
-    </collision>
-      <inertial>
-          <origin xyz="0 0 0" rpy="0.0 0.0 0.0"/>
-          <mass value="0.1"/>
-          <inertia ixx="0.1" ixy="0.0" ixz="0.0" iyy="0.1" iyz="0.0" izz="0.1"/>
-      </inertial>
-  </link>
-  <!-- Finger Joint 1 -->
-  <joint name="panda_finger_joint1" type="prismatic">
-    <parent link="panda_hand"/>
-    <child link="panda_leftfinger"/>
-    <origin rpy="0 0 0" xyz="0 0 0.0584"/>
-    <axis xyz="0 1 0"/>
-    <limit effort="30.0" lower="0.0" upper="0.04" velocity="10.0"/>
-  </joint>
-  <!-- Finger Joint 2 -->
-  <joint name="panda_finger_joint2" type="prismatic">
-    <parent link="panda_hand"/>
-    <child link="panda_rightfinger"/>
-    <origin rpy="0 0 0" xyz="0 0 0.0584"/>
-    <axis xyz="0 -1 0"/>
-    <limit effort="30.0" lower="0.0" upper="0.04" velocity="10.0"/>
-    <!-- <mimic joint="panda_finger_joint1" multiplier="-1"/> -->
+    <child link="panda_tool"/>
+    <origin rpy="0 0 0" xyz="0 0 0.106"/>
+  </joint>
+  <!-- TCP frame at the probe tip -->
+  <link name="panda_tcp"/>
+  <joint name="panda_tcp_joint" type="fixed">
+    <parent link="panda_tool"/>
+    <child link="panda_tcp"/>
+    <origin rpy="0 0 0" xyz="0 0 0.12"/>
   </joint>
 </robot>

File: panda_ws/src/panda_description/urdf/gazebo.xacro (robot description, xacro)
@@ -107,20 +107,4 @@
       <state_interface name="velocity"/>
     </joint>
-    <!-- Gripper Finger Joint 1 -->
-    <joint name="panda_finger_joint1">
-      <command_interface name="position">
-        <param name="min">0.0</param>
-        <param name="max">0.04</param>
-      </command_interface>
-      <state_interface name="position"/>
-    </joint>
-    <!-- Gripper Finger Joint 2 (Mimics Joint 1) -->
-    <joint name="panda_finger_joint2">
-      <command_interface name="position">
-        <param name="min">0.0</param>
-        <param name="max">0.04</param>
-      </command_interface>
-      <state_interface name="position"/>
-    </joint>
   </ros2_control>
 </robot>

Commit message: added a "LIDAR" sensor, to simulate a ray to measure distance

File: panda_ws/src/panda_description/urdf/arm.xacro (robot description, xacro)
@@ -260,4 +260,15 @@
     </inertial>
   </link>
+<gazebo reference="panda_tool">
+  <material>
+    <pbr>
+      <metal>
+        <albedo>0.7 0.7 0.75 1</albedo>
+        <metalness>1.0</metalness>
+        <roughness>0.2</roughness>
+      </metal>
+    </pbr>
+  </material>
+</gazebo>
   <!-- Tool joint at flange -->
   <joint name="panda_tool_joint" type="fixed">
@@ -267,5 +278,10 @@
   </joint>
   <!-- TCP frame at the probe tip -->
-  <link name="panda_tcp"/>
+  <link name="panda_tcp">
+    <inertial>
+      <mass value="0.01"/>
+      <inertia ixx="0.0001" ixy="0" ixz="0" iyy="0.0001" iyz="0" izz="0.0001"/>
+    </inertial>
+  </link>
   <joint name="panda_tcp_joint" type="fixed">
     <parent link="panda_tool"/>
@@ -273,3 +289,14 @@
     <origin rpy="0 0 0" xyz="0 0 0.12"/>
   </joint>
+  <link name="panda_lidar_frame">
+  <inertial>
+    <mass value="0.001"/>
+    <inertia ixx="0.00001" ixy="0" ixz="0" iyy="0.00001" iyz="0" izz="0.00001"/>
+  </inertial>
+</link>
+<joint name="panda_lidar_joint" type="fixed">
+  <parent link="panda_tcp"/>
+  <child link="panda_lidar_frame"/>
+  <origin rpy="0 -1.570796 0" xyz="0 0 0"/>
+</joint>
 </robot>

File: panda_ws/src/panda_description/urdf/sensors.xacro (robot description, xacro)
@@ -59,3 +59,28 @@
         </sensor>
   </gazebo>
+  <!-- Single-beam range sensor at TCP tip -->
+<gazebo reference="panda_lidar_frame">
+  <sensor name="probe_range" type="gpu_lidar">
+    <pose>0 0 0 0 0 0</pose> <always_on>true</always_on>
+    <update_rate>50</update_rate>
+    <visualize>true</visualize>
+    <topic>probe/scan</topic>
+    <gz_frame_id>panda_lidar_frame</gz_frame_id>
+    <lidar>
+      <scan>
+        <horizontal>
+          <samples>3</samples>
+          <resolution>1</resolution>
+          <min_angle>-0.01</min_angle>
+          <max_angle>0.01</max_angle>
+        </horizontal>
+      </scan>
+      <range>
+        <min>0.01</min>
+        <max>1.0</max>
+        <resolution>0.001</resolution>
+      </range>
+    </lidar>
+  </sensor>
+</gazebo>
 </robot>

Commit message: made the diameter of the tool smaller to represent a 25-gauge

File: panda_ws/src/panda_description/urdf/arm.xacro (robot description, xacro)
@@ -233,5 +233,5 @@
       <origin xyz="0 0 0.11" rpy="0 0 0"/>
       <geometry>
-        <cylinder radius="0.0008" length="0.02"/>
+        <cylinder radius="0.0005" length="0.02"/>
       </geometry>
     </visual>
@@ -251,5 +251,5 @@
       <origin xyz="0 0 0.11" rpy="0 0 0"/>
       <geometry>
-        <cylinder radius="0.0008" length="0.02"/>
+        <cylinder radius="0.0005" length="0.02"/>
       </geometry>
     </collision>
